Commit message: Add collisions

File: src/my_bot/description/robot_core.xacro (robot description, xacro)
@@ -19,4 +19,10 @@
             <material name="white" />
         </visual>
+        <collision>
+            <origin xyz="0.1 0 0.025" rpy="0 0 0" />
+            <geometry>
+                <box size="0.2 0.1 0.05" />
+            </geometry>
+        </collision>
     </link>
     <!-- LEFT WHEEL -->
@@ -34,4 +40,9 @@
             <material name="blue" />
         </visual>
+        <collision>
+            <geometry>
+                <cylinder radius="0.015" length="0.02" />
+            </geometry>
+        </collision>
     </link>
     <!-- RIGHT WHEEL -->
@@ -49,7 +60,12 @@
             <material name="blue" />
         </visual>
+        <collision>
+            <geometry>
+                <cylinder radius="0.015" length="0.02" />
+            </geometry>
+        </collision>
     </link>
     <!-- CASTER WHEELS -->
-    <joint name="front_caster_wheel_joint" type="continuous">
+    <joint name="front_caster_wheel_joint" type="fixed">
         <parent link="chassis" />
         <child link="front_caster_wheel" />
@@ -63,6 +79,11 @@
             <material name="black" />
         </visual>
+        <collision>
+            <geometry>
+                <sphere radius="0.0125" />
+            </geometry>
+        </collision>
     </link>
-    <joint name="rear_caster_wheel_joint" type="continuous">
+    <joint name="rear_caster_wheel_joint" type="fixed">
         <parent link="chassis" />
         <child link="rear_caster_wheel" />
@@ -76,4 +97,9 @@
             <material name="black" />
         </visual>
+        <collision>
+            <geometry>
+                <sphere radius="0.0125" />
+            </geometry>
+        </collision>
     </link>
 </robot>

Commit message: Add inertia

File: src/my_bot/description/robot_core.xacro (robot description, xacro)
@@ -2,4 +2,5 @@
 <robot xmlns:xacro="http://www.ros.org/wiki/xacro">
     <xacro:include filename="materials.xacro" />
+    <xacro:include filename="inertial_macros.xacro" />
     <link name="base">
     </link>
@@ -25,4 +26,7 @@
             </geometry>
         </collision>
+        <xacro:inertial_box mass="0.5" x="0.2" y="0.1" z="0.05">
+            <origin xyz="0.1 0 0.025" rpy="0 0 0" />
+        </xacro:inertial_box>
     </link>
     <!-- LEFT WHEEL -->
@@ -45,4 +49,7 @@
             </geometry>
         </collision>
+        <xacro:inertial_cylinder mass="0.1" radius="0.015" length="0.02">
+            <origin xyz="0 0 0" rpy="0 0 0" />
+        </xacro:inertial_cylinder>
     </link>
     <!-- RIGHT WHEEL -->
@@ -65,4 +72,7 @@
             </geometry>
         </collision>
+        <xacro:inertial_cylinder mass="0.1" radius="0.015" length="0.02">
+            <origin xyz="0 0 0" rpy="0 0 0" />
+        </xacro:inertial_cylinder>
     </link>
     <!-- CASTER WHEELS -->
@@ -84,4 +94,7 @@
             </geometry>
         </collision>
+        <xacro:inertial_sphere mass="0.05" radius="0.0125">
+            <origin xyz="0 0 0" rpy="0 0 0" />
+        </xacro:inertial_sphere>
     </link>
     <joint name="rear_caster_wheel_joint" type="fixed">
@@ -102,4 +115,7 @@
             </geometry>
         </collision>
+        <xacro:inertial_sphere mass="0.05" radius="0.0125">
+            <origin xyz="0 0 0" rpy="0 0 0" />
+        </xacro:inertial_sphere>
     </link>
 </robot>
