Commit message: Progress?

File: src/my_bot/description/robot.urdf.xacro (robot description, xacro)
@@ -1,5 +1,13 @@
 <?xml version="1.0"?>
 <robot xmlns:xacro="http://www.ros.org/wiki/xacro" name="robot">
+    <xacro:arg name="use_ros2_control" default="true" />
+    <xacro:arg name="sim_mode" default="false" />
     <xacro:include filename="robot_core.xacro" />
-    <xacro:include filename="gazebo_control.xacro" />
+    <xacro:include filename="ros2_control.xacro" />
+    <!-- <xacro:if value="$(arg use_ros2_control)">
+        <xacro:include filename="ros2_control.xacro" />
+    </xacro:if>
+    <xacro:unless value="$(arg use_ros2_control)">
+        <xacro:include filename="gazebo_control.xacro" />
+    </xacro:unless> -->
 </robot>

File: src/my_bot/description/robot_core.xacro (robot description, xacro)
@@ -3,9 +3,9 @@
     <xacro:include filename="materials.xacro" />
     <xacro:include filename="inertial_macros.xacro" />
-    <link name="base">
+    <link name="base_link">
     </link>
     <!-- BASE -->
     <joint name="base_to_chassis" type="fixed">
-        <parent link="base" />
+        <parent link="base_link" />
         <child link="chassis" />
         <origin xyz="-0.1 0 0" rpy="0 0 0" />
@@ -32,5 +32,5 @@
     <!-- LEFT WHEEL -->
     <joint name="left_wheel_joint" type="continuous">
-        <parent link="base" />
+        <parent link="base_link" />
         <child link="left_wheel" />
         <origin xyz="0 0.05 0" rpy="${-pi/2} 0 0" />
@@ -40,5 +40,5 @@
         <visual>
             <geometry>
-                <cylinder radius="0.015" length="0.02" />
+                <cylinder radius="0.05" length="0.02" />
             </geometry>
             <material name="blue" />
@@ -46,8 +46,8 @@
         <collision>
             <geometry>
-                <cylinder radius="0.015" length="0.02" />
+                <cylinder radius="0.05" length="0.02" />
             </geometry>
         </collision>
-        <xacro:inertial_cylinder mass="0.1" radius="0.015" length="0.02">
+        <xacro:inertial_cylinder mass="0.1" radius="0.05" length="0.02">
             <origin xyz="0 0 0" rpy="0 0 0" />
         </xacro:inertial_cylinder>
@@ -55,5 +55,5 @@
     <!-- RIGHT WHEEL -->
     <joint name="right_wheel_joint" type="continuous">
-        <parent link="base" />
+        <parent link="base_link" />
         <child link="right_wheel" />
         <origin xyz="0 -0.05 0" rpy="${pi/2} 0 0" />
@@ -63,5 +63,5 @@
         <visual>
             <geometry>
-                <cylinder radius="0.015" length="0.02" />
+                <cylinder radius="0.05" length="0.02" />
             </geometry>
             <material name="blue" />
@@ -69,8 +69,8 @@
         <collision>
             <geometry>
-                <cylinder radius="0.015" length="0.02" />
+                <cylinder radius="0.05" length="0.02" />
             </geometry>
         </collision>
-        <xacro:inertial_cylinder mass="0.1" radius="0.015" length="0.02">
+        <xacro:inertial_cylinder mass="0.1" radius="0.05" length="0.02">
             <origin xyz="0 0 0" rpy="0 0 0" />
         </xacro:inertial_cylinder>
